Commit message: .

File: iiwa_ros/iiwa_description/urdf/iiwa14.xacro (robot description, xacro)
@@ -30,5 +30,5 @@
   <!-- some constants -->
   <xacro:property name="safety_controller_k_pos" value="100"/>
-  <xacro:property name="safety_controller_k_vel" value="2"/>
+  <xacro:property name="safety_controller_k_vel" value="10"/>
   <xacro:property name="safety_percentage" value="0.95"/>
   <xacro:property name="joint_damping" value="0.5"/>

File: iiwa_ros/iiwa_description/urdf/iiwa7.xacro (robot description, xacro)
@@ -55,6 +55,6 @@
   <xacro:property name="max_velocity_4" value="${130 * PI / 180.}"/>
   <xacro:property name="max_velocity_5" value="${140 * PI / 180.}"/>
-  <xacro:property name="max_velocity_6" value="${PI}"/>
-  <xacro:property name="max_velocity_7" value="${PI}"/>
+  <xacro:property name="max_velocity_6" value="${PI/2}"/>
+  <xacro:property name="max_velocity_7" value="${PI/2}"/>
   <xacro:macro name="iiwa7" params="parent hardware_interface robot_name collision_postfix *origin">
     <!--joint between {parent} and link_0-->
